Commit message: adding humble ign version

File: lbr_description/gazebo/lbr_gazebo.xacro (robot description, xacro)
@@ -4,11 +4,8 @@
         <!-- ros_control-plugin -->
         <gazebo>
-            <plugin name="gazebo_ros2_control" filename="libgazebo_ros2_control.so">
+            <plugin filename="ign_ros2_control-system"
+                name="ign_ros2_control::IgnitionROS2ControlPlugin">
                 <parameters>$(find lbr_ros2_control)/config/lbr_controllers.yaml</parameters>
-                <ros>
-                    <namespace>/${robot_name}</namespace>
-                    <!-- remapping for controller manager inside Gazebo plugin -->
-                    <remapping>~/robot_description:=robot_description</remapping>
-                </ros>
+                <remapping>~/robot_description:=robot_description</remapping>
             </plugin>
         </gazebo>

File: lbr_description/urdf/med14/med14_description.xacro (robot description, xacro)
@@ -31,5 +31,5 @@
                 <origin rpy="0 0 0" xyz="0 0 0" />
                 <geometry>
-                    <mesh filename="package://lbr_description/meshes/med14/visual/link_0.dae" />
+                    <mesh filename="file://$(find lbr_description)/meshes/med14/visual/link_0.dae" />
                 </geometry>
             </visual>
@@ -37,5 +37,5 @@
                 <origin rpy="0 0 0" xyz="0 0 0" />
                 <geometry>
-                    <mesh filename="package://lbr_description/meshes/med14/collision/link_0.stl" />
+                    <mesh filename="file://$(find lbr_description)/meshes/med14/collision/link_0.stl" />
                 </geometry>
             </collision>
@@ -63,5 +63,5 @@
                 <origin rpy="0 0 0" xyz="0.0 0.0 -0.147" />
                 <geometry>
-                    <mesh filename="package://lbr_description/meshes/med14/visual/link_1.dae" />
+                    <mesh filename="file://$(find lbr_description)/meshes/med14/visual/link_1.dae" />
                 </geometry>
             </visual>
@@ -69,5 +69,5 @@
                 <origin rpy="0 0 0" xyz="0.0 0.0 -0.147" />
                 <geometry>
-                    <mesh filename="package://lbr_description/meshes/med14/collision/link_1.stl" />
+                    <mesh filename="file://$(find lbr_description)/meshes/med14/collision/link_1.stl" />
                 </geometry>
             </collision>
@@ -95,5 +95,5 @@
                 <origin rpy="0 0 0" xyz="0.0 0.01 -0.3595" />
                 <geometry>
-                    <mesh filename="package://lbr_description/meshes/med14/visual/link_2.dae" />
+                    <mesh filename="file://$(find lbr_description)/meshes/med14/visual/link_2.dae" />
                 </geometry>
             </visual>
@@ -101,5 +101,5 @@
                 <origin rpy="0 0 0" xyz="0.0 0.01 -0.3595" />
                 <geometry>
-                    <mesh filename="package://lbr_description/meshes/med14/collision/link_2.stl" />
+                    <mesh filename="file://$(find lbr_description)/meshes/med14/collision/link_2.stl" />
                 </geometry>
             </collision>
@@ -127,5 +127,5 @@
                 <origin rpy="0 0 0" xyz="0.0 0.0 -0.5875" />
                 <geometry>
-                    <mesh filename="package://lbr_description/meshes/med14/visual/link_3.dae" />
+                    <mesh filename="file://$(find lbr_description)/meshes/med14/visual/link_3.dae" />
                 </geometry>
             </visual>
@@ -133,5 +133,5 @@
                 <origin rpy="0 0 0" xyz="0.0 0.0 -0.5875" />
                 <geometry>
-                    <mesh filename="package://lbr_description/meshes/med14/collision/link_3.stl" />
+                    <mesh filename="file://$(find lbr_description)/meshes/med14/collision/link_3.stl" />
                 </geometry>
             </collision>
@@ -159,5 +159,5 @@
                 <origin rpy="0 0 0" xyz="0.0 -0.0105 -0.7795" />
                 <geometry>
-                    <mesh filename="package://lbr_description/meshes/med14/visual/link_4.dae" />
+                    <mesh filename="file://$(find lbr_description)/meshes/med14/visual/link_4.dae" />
                 </geometry>
             </visual>
@@ -165,5 +165,5 @@
                 <origin rpy="0 0 0" xyz="0.0 -0.0105 -0.7795" />
                 <geometry>
-                    <mesh filename="package://lbr_description/meshes/med14/collision/link_4.stl" />
+                    <mesh filename="file://$(find lbr_description)/meshes/med14/collision/link_4.stl" />
                 </geometry>
             </collision>
@@ -191,5 +191,5 @@
                 <origin rpy="0 0 0" xyz="0.0 0.0 -0.987" />
                 <geometry>
-                    <mesh filename="package://lbr_description/meshes/med14/visual/link_5.dae" />
+                    <mesh filename="file://$(find lbr_description)/meshes/med14/visual/link_5.dae" />
                 </geometry>
             </visual>
@@ -197,5 +197,5 @@
                 <origin rpy="0 0 0" xyz="0.0 0.0 -0.987" />
                 <geometry>
-                    <mesh filename="package://lbr_description/meshes/med14/collision/link_5.stl" />
+                    <mesh filename="file://$(find lbr_description)/meshes/med14/collision/link_5.stl" />
                 </geometry>
             </collision>
@@ -223,5 +223,5 @@
                 <origin rpy="0 0 0" xyz="0.0 0.0707 -1.1795" />
                 <geometry>
-                    <mesh filename="package://lbr_description/meshes/med14/visual/link_6.dae" />
+                    <mesh filename="file://$(find lbr_description)/meshes/med14/visual/link_6.dae" />
                 </geometry>
             </visual>
@@ -229,5 +229,5 @@
                 <origin rpy="0 0 0" xyz="0.0 0.0707 -1.1795" />
                 <geometry>
-                    <mesh filename="package://lbr_description/meshes/med14/collision/link_6.stl" />
+                    <mesh filename="file://$(find lbr_description)/meshes/med14/collision/link_6.stl" />
                 </geometry>
             </collision>
@@ -254,5 +254,5 @@
                 <origin rpy="0 0 0" xyz="0.0 0.0 -1.2705" />
                 <geometry>
-                    <mesh filename="package://lbr_description/meshes/med14/visual/link_7.dae" />
+                    <mesh filename="file://$(find lbr_description)/meshes/med14/visual/link_7.dae" />
                 </geometry>
             </visual>
@@ -260,5 +260,5 @@
                 <origin rpy="0 0 0" xyz="0.0 0.0 -1.2705" />
                 <geometry>
-                    <mesh filename="package://lbr_description/meshes/med14/collision/link_7.stl" />
+                    <mesh filename="file://$(find lbr_description)/meshes/med14/collision/link_7.stl" />
                 </geometry>
             </collision>

File: lbr_ros2_control/config/lbr_system_interface.xacro (robot description, xacro)
@@ -15,5 +15,5 @@
             <xacro:if value="${mode == 'gazebo'}">
                 <hardware>
-                    <plugin>gazebo_ros2_control/GazeboSystem</plugin>
+                    <plugin>ign_ros2_control/IgnitionSystem</plugin>
                 </hardware>
             </xacro:if>
@@ -94,8 +94,4 @@
                         <param name="max">${max_position}</param>
                     </command_interface>
-                    <command_interface name="effort">
-                        <param name="min">-${max_torque}</param>
-                        <param name="max"> ${max_torque}</param>
-                    </command_interface>
                     <state_interface name="position" />
                     <state_interface name="velocity" />

Commit message: tested in rviz and ign gz OK

File: lbr_description/gazebo/lbr_gazebo.xacro (robot description, xacro)
@@ -6,5 +6,10 @@
             <plugin filename="ign_ros2_control-system" name="ign_ros2_control::IgnitionROS2ControlPlugin">
                 <parameters>$(find lbr_ros2_control)/config/lbr_controllers.yaml</parameters>
-                <remapping>~/robot_description:=robot_description</remapping>
+                <robot_param_node>robot_state_publisher</robot_param_node>
+                <robot_param_node>robot_description</robot_param_node>
+                <ros>
+                    <namespace>/${robot_name}</namespace>
+                    <remapping>~/robot_description:=robot_description</remapping>
+                </ros>
             </plugin>
         </gazebo>

File: lbr_description/urdf/iiwa14/iiwa14_description.xacro (robot description, xacro)
@@ -31,5 +31,5 @@
                 <origin rpy="0 0 0" xyz="0 0 0" />
                 <geometry>
-                    <mesh filename="package://lbr_description/meshes/iiwa14/visual/link_0.dae" />
+                    <mesh filename="file://$(find lbr_description)/meshes/iiwa14/visual/link_0.dae" />
                 </geometry>
             </visual>
@@ -37,5 +37,5 @@
                 <origin rpy="0 0 0" xyz="0 0 0" />
                 <geometry>
-                    <mesh filename="package://lbr_description/meshes/iiwa14/collision/link_0.stl" />
+                    <mesh filename="file://$(find lbr_description)/meshes/iiwa14/collision/link_0.stl" />
                 </geometry>
             </collision>
@@ -63,5 +63,5 @@
                 <origin rpy="0 0 0" xyz="0.0 0.0 -0.1475" />
                 <geometry>
-                    <mesh filename="package://lbr_description/meshes/iiwa14/visual/link_1.dae" />
+                    <mesh filename="file://$(find lbr_description)/meshes/iiwa14/visual/link_1.dae" />
                 </geometry>
             </visual>
@@ -69,5 +69,5 @@
                 <origin rpy="0 0 0" xyz="0.0 0.0 -0.1475" />
                 <geometry>
-                    <mesh filename="package://lbr_description/meshes/iiwa14/collision/link_1.stl" />
+                    <mesh filename="file://$(find lbr_description)/meshes/iiwa14/collision/link_1.stl" />
                 </geometry>
             </collision>
@@ -95,5 +95,5 @@
                 <origin rpy="0 0 0" xyz="0.0 0.01 -0.36" />
                 <geometry>
-                    <mesh filename="package://lbr_description/meshes/iiwa14/visual/link_2.dae" />
+                    <mesh filename="file://$(find lbr_description)/meshes/iiwa14/visual/link_2.dae" />
                 </geometry>
             </visual>
@@ -101,5 +101,5 @@
                 <origin rpy="0 0 0" xyz="0.0 0.01 -0.36" />
                 <geometry>
-                    <mesh filename="package://lbr_description/meshes/iiwa14/collision/link_2.stl" />
+                    <mesh filename="file://$(find lbr_description)/meshes/iiwa14/collision/link_2.stl" />
                 </geometry>
             </collision>
@@ -127,5 +127,5 @@
                 <origin rpy="0 0 0" xyz="0.0 0.0 -0.588" />
                 <geometry>
-                    <mesh filename="package://lbr_description/meshes/iiwa14/visual/link_3.dae" />
+                    <mesh filename="file://$(find lbr_description)/meshes/iiwa14/visual/link_3.dae" />
                 </geometry>
             </visual>
@@ -133,5 +133,5 @@
                 <origin rpy="0 0 0" xyz="0.0 0.0 -0.588" />
                 <geometry>
-                    <mesh filename="package://lbr_description/meshes/iiwa14/collision/link_3.stl" />
+                    <mesh filename="file://$(find lbr_description)/meshes/iiwa14/collision/link_3.stl" />
                 </geometry>
             </collision>
@@ -159,5 +159,5 @@
                 <origin rpy="0 0 0" xyz="0.0 -0.0105 -0.78" />
                 <geometry>
-                    <mesh filename="package://lbr_description/meshes/iiwa14/visual/link_4.dae" />
+                    <mesh filename="file://$(find lbr_description)/meshes/iiwa14/visual/link_4.dae" />
                 </geometry>
             </visual>
@@ -165,5 +165,5 @@
                 <origin rpy="0 0 0" xyz="0.0 -0.0105 -0.78" />
                 <geometry>
-                    <mesh filename="package://lbr_description/meshes/iiwa14/collision/link_4.stl" />
+                    <mesh filename="file://$(find lbr_description)/meshes/iiwa14/collision/link_4.stl" />
                 </geometry>
             </collision>
@@ -191,5 +191,5 @@
                 <origin rpy="0 0 0" xyz="0.0 0.0 -0.9875" />
                 <geometry>
-                    <mesh filename="package://lbr_description/meshes/iiwa14/visual/link_5.dae" />
+                    <mesh filename="file://$(find lbr_description)/meshes/iiwa14/visual/link_5.dae" />
                 </geometry>
             </visual>
@@ -197,5 +197,5 @@
                 <origin rpy="0 0 0" xyz="0.0 0.0 -0.9875" />
                 <geometry>
-                    <mesh filename="package://lbr_description/meshes/iiwa14/collision/link_5.stl" />
+                    <mesh filename="file://$(find lbr_description)/meshes/iiwa14/collision/link_5.stl" />
                 </geometry>
             </collision>
@@ -223,5 +223,5 @@
                 <origin rpy="0 0 0" xyz="0.0 0.0707 -1.18" />
                 <geometry>
-                    <mesh filename="package://lbr_description/meshes/iiwa14/visual/link_6.dae" />
+                    <mesh filename="file://$(find lbr_description)/meshes/iiwa14/visual/link_6.dae" />
                 </geometry>
             </visual>
@@ -229,5 +229,5 @@
                 <origin rpy="0 0 0" xyz="0.0 0.0707 -1.18" />
                 <geometry>
-                    <mesh filename="package://lbr_description/meshes/iiwa14/collision/link_6.stl" />
+                    <mesh filename="file://$(find lbr_description)/meshes/iiwa14/collision/link_6.stl" />
                 </geometry>
             </collision>
@@ -254,5 +254,5 @@
                 <origin rpy="0 0 0" xyz="0.0 0.0 -1.271" />
                 <geometry>
-                    <mesh filename="package://lbr_description/meshes/iiwa14/visual/link_7.dae" />
+                    <mesh filename="file://$(find lbr_description)/meshes/iiwa14/visual/link_7.dae" />
                 </geometry>
             </visual>
@@ -260,5 +260,5 @@
                 <origin rpy="0 0 0" xyz="0.0 0.0 -1.271" />
                 <geometry>
-                    <mesh filename="package://lbr_description/meshes/iiwa14/collision/link_7.stl" />
+                    <mesh filename="file://$(find lbr_description)/meshes/iiwa14/collision/link_7.stl" />
                 </geometry>
             </collision>

File: lbr_description/urdf/med7/med7_description.xacro (robot description, xacro)
@@ -32,5 +32,5 @@
                 <origin rpy="0 0 0" xyz="0 0 0" />
                 <geometry>
-                    <mesh filename="package://lbr_description/meshes/med7/visual/link_0.dae" />
+                    <mesh filename="file://$(find lbr_description)/meshes/med7/visual/link_0.dae" />
                 </geometry>
             </visual>
@@ -38,5 +38,5 @@
                 <origin rpy="0 0 0" xyz="0 0 0" />
                 <geometry>
-                    <mesh filename="package://lbr_description/meshes/med7/collision/link_0.stl" />
+                    <mesh filename="file://$(find lbr_description)/meshes/med7/collision/link_0.stl" />
                 </geometry>
             </collision>
@@ -64,5 +64,5 @@
                 <origin rpy="0 0 0" xyz="0.0 0.0 -0.1475" />
                 <geometry>
-                    <mesh filename="package://lbr_description/meshes/med7/visual/link_1.dae" />
+                    <mesh filename="file://$(find lbr_description)/meshes/med7/visual/link_1.dae" />
                 </geometry>
             </visual>
@@ -70,5 +70,5 @@
                 <origin rpy="0 0 0" xyz="0.0 0.0 -0.1475" />
                 <geometry>
-                    <mesh filename="package://lbr_description/meshes/med7/collision/link_1.stl" />
+                    <mesh filename="file://$(find lbr_description)/meshes/med7/collision/link_1.stl" />
                 </geometry>
             </collision>
@@ -96,5 +96,5 @@
                 <origin rpy="0 0 0" xyz="0.0 0.0105 -0.34" />
                 <geometry>
-                    <mesh filename="package://lbr_description/meshes/med7/visual/link_2.dae" />
+                    <mesh filename="file://$(find lbr_description)/meshes/med7/visual/link_2.dae" />
                 </geometry>
             </visual>
@@ -102,5 +102,5 @@
                 <origin rpy="0 0 0" xyz="0.0 0.0105 -0.34" />
                 <geometry>
-                    <mesh filename="package://lbr_description/meshes/med7/collision/link_2.stl" />
+                    <mesh filename="file://$(find lbr_description)/meshes/med7/collision/link_2.stl" />
                 </geometry>
             </collision>
@@ -128,5 +128,5 @@
                 <origin rpy="0 0 0" xyz="0.0 0.0 -0.5475" />
                 <geometry>
-                    <mesh filename="package://lbr_description/meshes/med7/visual/link_3.dae" />
+                    <mesh filename="file://$(find lbr_description)/meshes/med7/visual/link_3.dae" />
                 </geometry>
             </visual>
@@ -134,5 +134,5 @@
                 <origin rpy="0 0 0" xyz="0.0 0.0 -0.5475" />
                 <geometry>
-                    <mesh filename="package://lbr_description/meshes/med7/collision/link_3.stl" />
+                    <mesh filename="file://$(find lbr_description)/meshes/med7/collision/link_3.stl" />
                 </geometry>
             </collision>
@@ -160,5 +160,5 @@
                 <origin rpy="0 0 0" xyz="0.0 -0.0105 -0.74" />
                 <geometry>
-                    <mesh filename="package://lbr_description/meshes/med7/visual/link_4.dae" />
+                    <mesh filename="file://$(find lbr_description)/meshes/med7/visual/link_4.dae" />
                 </geometry>
             </visual>
@@ -166,5 +166,5 @@
                 <origin rpy="0 0 0" xyz="0.0 -0.0105 -0.74" />
                 <geometry>
-                    <mesh filename="package://lbr_description/meshes/med7/collision/link_4.stl" />
+                    <mesh filename="file://$(find lbr_description)/meshes/med7/collision/link_4.stl" />
                 </geometry>
             </collision>
@@ -192,5 +192,5 @@
                 <origin rpy="0 0 0" xyz="0.0 0.0 -0.9475" />
                 <geometry>
-                    <mesh filename="package://lbr_description/meshes/med7/visual/link_5.dae" />
+                    <mesh filename="file://$(find lbr_description)/meshes/med7/visual/link_5.dae" />
                 </geometry>
             </visual>
@@ -198,5 +198,5 @@
                 <origin rpy="0 0 0" xyz="0.0 0.0 -0.9475" />
                 <geometry>
-                    <mesh filename="package://lbr_description/meshes/med7/collision/link_5.stl" />
+                    <mesh filename="file://$(find lbr_description)/meshes/med7/collision/link_5.stl" />
                 </geometry>
             </collision>
@@ -224,5 +224,5 @@
                 <origin rpy="0 0 0" xyz="0.0 0.0707 -1.14" />
                 <geometry>
-                    <mesh filename="package://lbr_description/meshes/med7/visual/link_6.dae" />
+                    <mesh filename="file://$(find lbr_description)/meshes/med7/visual/link_6.dae" />
                 </geometry>
             </visual>
@@ -230,5 +230,5 @@
                 <origin rpy="0 0 0" xyz="0.0 0.0707 -1.14" />
                 <geometry>
-                    <mesh filename="package://lbr_description/meshes/med7/collision/link_6.stl" />
+                    <mesh filename="file://$(find lbr_description)/meshes/med7/collision/link_6.stl" />
                 </geometry>
             </collision>
@@ -255,5 +255,5 @@
                 <origin rpy="0 0 0" xyz="0.0 0.0 -1.231" />
                 <geometry>
-                    <mesh filename="package://lbr_description/meshes/med7/visual/link_7.dae" />
+                    <mesh filename="file://$(find lbr_description)/meshes/med7/visual/link_7.dae" />
                 </geometry>
             </visual>
@@ -261,5 +261,5 @@
                 <origin rpy="0 0 0" xyz="0.0 0.0 -1.231" />
                 <geometry>
-                    <mesh filename="package://lbr_description/meshes/med7/collision/link_7.stl" />
+                    <mesh filename="file://$(find lbr_description)/meshes/med7/collision/link_7.stl" />
                 </geometry>
             </collision>

File: lbr_ros2_control/config/lbr_system_interface.xacro (robot description, xacro)
@@ -15,5 +15,5 @@
             <xacro:if value="${mode == 'gazebo'}">
                 <hardware>
-                    <plugin>mock_components/GenericSystem</plugin>
+                    <plugin>ign_ros2_control/IgnitionSystem</plugin>
                 </hardware>
             </xacro:if>
