Commit message: added zed setup for interim needs

File: lbr_description/urdf/med14/med14_description.xacro (robot description, xacro)
@@ -7,4 +7,7 @@
         <xacro:include filename="$(find lbr_description)/gazebo/lbr_gazebo.xacro" />
         <xacro:include filename="$(find lbr_ros2_control)/config/lbr_system_interface.xacro" />
+        <!-- Include the ZED camera macro -->
+        <xacro:include filename="$(find lbr_description)/urdf/zed/zed_macro.urdf.xacro" />
+        <xacro:zed_camera name="zedm" model="zedm"/>
         <!-- joint limits via yaml -->
         <xacro:property name="joint_limits_path"
@@ -271,4 +274,28 @@
         <link name="link_ee">
         </link>
+                <joint name="joint_mount" type="fixed">
+            <origin rpy="0 3.145 0" xyz="0.0 0.0 -0.01" />
+            <parent link="link_ee" />
+            <child link="mount" />
+        </joint>
+        <link name="mount">
+            <visual>
+                <origin rpy="0.0 0 0" xyz="0.0 0.0 0.0" />
+                <geometry>
+                    <mesh filename="file://$(find lbr_description)/meshes/mount/Kuka_Scanner_mount_4.dae" />
+                </geometry>
+            </visual>
+            <collision>
+                <origin rpy="0 0 0" xyz="0.0 0.0 0.0" />
+                <geometry>
+                    <mesh filename="file://$(find lbr_description)/meshes/mount/Kuka_Scanner_mount_4.dae" />
+                </geometry>
+            </collision>
+        </link>
+        <joint name="zedm_joint" type="fixed">
+            <parent link="mount"/>
+            <child link="zedm_camera_link"/>
+            <origin xyz="0.007 ${100/1000} ${-95/1000}" rpy="0.0 ${135*3.145/180.0} ${3.145/2.0}"/>
+        </joint>
     </xacro:macro>
 </robot>

Commit message: added material to the ee mount

File: lbr_description/urdf/med14/med14_description.xacro (robot description, xacro)
@@ -285,4 +285,7 @@
                     <mesh filename="file://$(find lbr_description)/meshes/mount/Kuka_Scanner_mount_4.dae" />
                 </geometry>
+                <material name="zed2_mat">
+                    <color rgba="0.25 0.25 0.25 1.0"/>
+                </material>
             </visual>
             <collision>

Commit message: updated get_eef_pose

File: lbr_description/urdf/med14/med14_description.xacro (robot description, xacro)
@@ -9,5 +9,7 @@
         <!-- Include the ZED camera macro -->
         <xacro:include filename="$(find zed_wrapper)/urdf/zed_macro.urdf.xacro" />
-        <xacro:zed_camera name="zedm" model="zedm"/>
+        <xacro:zed_camera name="zedm" >
+            <gnss_origin/>
+        </xacro:zed_camera>
         <!-- joint limits via yaml -->
         <xacro:property name="joint_limits_path"
@@ -274,5 +276,5 @@
         <link name="link_ee">
         </link>
-                <joint name="joint_mount" type="fixed">
+        <joint name="joint_mount" type="fixed">
             <origin rpy="0 3.145 0" xyz="0.0 0.0 -0.01" />
             <parent link="link_ee" />

File: lbr_ros2_control/config/lbr_system_interface.xacro (robot description, xacro)
@@ -90,10 +90,11 @@
                 params="name min_position max_position max_velocity max_torque mode">
                 <joint name="${name}">
-                    <!-- <command_interface name="position">
+                    <command_interface name="position">
                         <param name="min">${min_position}</param>
                         <param name="max">${max_position}</param>
-                    </command_interface> -->
-                    <command_interface name="velocity">
-                        <param name="max"> ${max_velocity}</param>
+                    </command_interface>
+                    <command_interface name="effort">
+                        <param name="min"> ${max_torque}</param>
+                        <param name="max"> ${max_torque}</param>
                     </command_interface>
                     <state_interface name="position" />
